File: amp/amp.kicad_sch (KiCad schematic)
At the start: 0 parts

Commit message: WIP schematic
Parts:
- added C1, C5, C8: 10nF, symbol Device:C
- added C2, C4: 2.2uF, symbol Device:C_Polarized
- added C3: 1nF, symbol Device:C
- added C6, C9: 100nF, symbol Device:C
- added C7: 220uF, symbol Device:C_Polarized
- added J1: Input, symbol Connector_Audio:AudioJack2
- added J2: Speaker, symbol Connector_Audio:AudioJack2
- added R1, R2, R3, R4, R6, R9: 1M, symbol Device:R
- added R10, R7: 100, symbol Device:R
- added R11, R8: 220K, symbol Device:R
- added R12: 47, symbol Device:R
- added R13, R14: 10K, symbol Device:R
- added R5: 47K, symbol Device:R
- added RV1: 500k log, symbol Device:R_Potentiometer
- added RV2: 50k log, symbol Device:R_Potentiometer
- added U1: NE5532, symbol Amplifier_Operational:NE5532
- added U2: ECC83, Valve:Valve_Noval_P, symbol Valve:ECC83
- added U3: LM386, symbol Amplifier_Audio:LM386
Connections:
- new net: C1.2, R1.2, U1.3 (+)
- new net: C2.1, R2.1
- new net: R7.2, U2.8 (K)
- new net: R2.2, RV1.1, U1.2 (-)
- new net: C7.2, J2.T
- new net: C6.1, R11.1, U2.1 (A)
- new net: C6.2, RV2.1
- new net: R10.2, U2.3 (K)
- new net: R13.1, R14.2, U1.5 (+)
- new net: RV2.2, U3.2 (-)
- new net: C7.1, C8.2, U3.5
- new net: C9.2, U3.7 (BYPASS)
- new net: C5.1, R8.1, U2.6 (A)
- new net: C1.1, J1.T
- new net: C3.2, R5.2, R6.2
- new net: U1.6 (-), U1.7
- new net: C3.1, RV1.2, U1.1
- new net: R5.1, U2.7 (G)
- new net: C5.2, R9.2, U2.2 (G)
- new net: C8.1, R12.2
- new net +12V: R11.2, R13.2, R4.2, R8.2, U1.8 (V+), U2.4 (F1), U3.6 (V+)
- new net +6V bias: C4.1, R1.1, R3.2, R4.1
- new net GND: C2.2, C4.2, C9.1, J1.S, J2.S, R10.1, R12.1, R14.1, R3.1, R6.1, R7.1, R9.1, RV2.3, U1.4 (V-), U2.5 (F1), U3.3 (+), U3.4 (GND)
- no-connect marks 0 -> 4
Other:
- note added: "Zobel"
